Commit message: Final  demo

File: easy_simulation/urdf/kinova_g3l_box_picker.urdf.xacro (robot description, xacro)
@@ -78,4 +78,7 @@
       name="camera"
       prefix="$(arg prefix)"/>
+    <xacro:gz_rgbd_camera_tiny
+      name="camera_hand"
+      prefix="$(arg prefix)"/>
   </xacro:if>
   <!-- RGBD camera URDF inclusion -->
@@ -84,6 +87,12 @@
     name="camera"
     prefix="$(arg prefix)">
-    <origin xyz="0.2 0 1.4" rpy="0 1.4 0"/>
+    <origin xyz="0.2 0 1.4" rpy="0 1.45 0"/>
   </xacro:rgbd_camera>
+  <xacro:rgbd_camera_tiny
+    parent_link="$(arg prefix)upper_wrist_link"
+    name="camera_hand"
+    prefix="$(arg prefix)">
+    <origin xyz="-0.1 0 0.08" rpy="0 3.0 0"/>
+  </xacro:rgbd_camera_tiny>
   <!-- Suction gripper URDF inclusion -->
   <xacro:include filename="$(find easy_simulation)/urdf/suction_gripper.urdf.xacro" />

File: easy_simulation/urdf/rgbd_camera.urdf.xacro (robot description, xacro)
@@ -23,4 +23,7 @@
             </visual>
         </link>
+        <gazebo reference="${prefix}${name}_frame">
+            <material>DarkGray</material>
+        </gazebo>
         <!-- Fixed joint connecting camera to parent -->
         <joint name="${prefix}${name}_joint" type="fixed">
@@ -100,3 +103,103 @@
         </gazebo>
     </xacro:macro>
+    <xacro:macro name="rgbd_camera_tiny" params="parent_link name prefix *origin">
+        <!-- Camera link -->
+        <link name="${prefix}${name}_frame">
+            <visual>
+                <geometry>
+                    <box size="0.015 0.03 0.03"/>
+                </geometry>
+                <material name="dark_gray">
+                    <ambient>0.05 0.05 0.05 1</ambient>
+                    <diffuse>0.05 0.05 0.05 1</diffuse>
+                    <specular>0.01 0.01 0.01 1</specular>
+                    <pbr type="metal">
+                        <albedo>0.05 0.05 0.05 1</albedo>
+                        <metalness>0.2</metalness>
+                        <roughness>0.9</roughness>
+                    </pbr>
+                </material>
+            </visual>
+        </link>
+        <gazebo reference="${prefix}${name}_frame">
+            <material>DarkGray</material>
+        </gazebo>
+        <!-- Fixed joint connecting camera to parent -->
+        <joint name="${prefix}${name}_joint" type="fixed">
+            <parent link="${parent_link}" />
+            <child link="${prefix}${name}_frame" />
+            <xacro:insert_block name="origin" />
+        </joint>
+        <link name="${prefix}${name}_optical_frame" />
+        <joint name="${prefix}${name}_optical_joint" type="fixed">
+            <parent link="${prefix}${name}_frame" />
+            <child link="${prefix}${name}_optical_frame" />
+            <origin xyz="0 0 0" rpy="-1.5708 0 -1.5708" />
+        </joint>
+    </xacro:macro>
+    <xacro:macro name="gz_rgbd_camera_tiny" params="name prefix">
+        <gazebo reference="${prefix}${name}_frame">
+            <sensor name="camera_sensor" type="rgbd_camera">
+                <camera>
+                    <horizontal_fov>1.8</horizontal_fov>
+                    <vertical_fov>1.8</vertical_fov>
+                    <image>
+                        <width>$(arg camera_width)</width>
+                        <height>$(arg camera_height)</height>
+                        <format>RGB_INT8</format>
+                    </image>
+                    <clip>
+                        <near>0.1</near>
+                        <far>5</far>
+                    </clip>
+                    <distortion>
+                        <k1>0.0</k1>
+                        <k2>0.0</k2>
+                        <k3>0.0</k3>
+                        <p1>0.0</p1>
+                        <p2>0.0</p2>
+                        <center>0.5 0.5</center>
+                    </distortion>
+                    <lens>
+                        <intrinsics>
+                            <fx>554.25469</fx>
+                            <fy>554.25469</fy>
+                            <cx>320.5</cx>
+                            <cy>240.5</cy>
+                            <s>0</s>
+                        </intrinsics>
+                        <!-- These need to match the intrinsics above or
+                    Gazebo will default to different default values -->
+                        <projection>
+                            <p_fx>554.25469</p_fx>
+                            <p_fy>554.25469</p_fy>
+                            <p_cx>320.5</p_cx>
+                            <p_cy>240.5</p_cy>
+                            <tx>0</tx>
+                            <ty>0</ty>
+                        </projection>
+                    </lens>
+                    <noise>
+                        <type>gaussian</type>
+                        <mean>0.003</mean>
+                        <stddev>0.005</stddev>
+                    </noise>
+                    <depth_camera>
+                        <clip>
+                            <near>0.25</near>
+                            <far>5</far>
+                        </clip>
+                    </depth_camera>
+                    <optical_frame_id>${prefix}${name}_optical_frame</optical_frame_id>
+                    <depth_frame_id>${prefix}${name}_depth_frame</depth_frame_id>
+                </camera>
+                <gz_frame_id>${prefix}${name}_frame</gz_frame_id>
+                <always_on>1</always_on>
+                <update_rate>$(arg camera_fps)</update_rate>
+                <visualize>true</visualize>
+                <topic>${prefix}${name}</topic>
+                <enable_metrics>false</enable_metrics>
+            </sensor>
+        </gazebo>
+    </xacro:macro>
 </robot>
