Commit message: Pick 80 percent, place 95 percent

File: easy_simulation/worlds/box_picking_desk.sdf.xacro (robot description, xacro)
@@ -86,380 +86,194 @@
       <self_collide>false</self_collide>
     </model>
-    <model name='Table'>
-      <static>true</static>
-      <link name='link'>
-        <collision name='surface'>
-          <pose>0 0 1 0 0 0</pose>
-          <geometry>
-            <box>
-              <size>1.5 0.80000000000000004 0.029999999999999999</size>
-            </box>
-          </geometry>
-          <surface>
-            <friction>
-              <ode>
-                <mu>0.59999999999999998</mu>
-                <mu2>0.59999999999999998</mu2>
-              </ode>
-            </friction>
-            <bounce />
-            <contact />
-          </surface>
-        </collision>
-        <visual name='visual1'>
-          <pose>0 0 1 0 0 0</pose>
-          <geometry>
-            <box>
-              <size>1.5 0.80000000000000004 0.029999999999999999</size>
-            </box>
-          </geometry>
-          <material>
-            <diffuse>1 1 1 1</diffuse>
-            <script>
+    <xacro:macro name="desk" params="name origin L W H">
+      <model name='${name}'>
+        <static>true</static>
+        <link name='link'>
+          <collision name='surface'>
+            <pose>0 0 ${H} 0 0 0</pose>
+            <geometry>
+              <box>
+                <size>${L} ${W} 0.03</size>
+              </box>
+            </geometry>
+            <surface>
+              <friction>
+                <ode>
+                  <mu>0.59999999999999998</mu>
+                  <mu2>0.59999999999999998</mu2>
+                </ode>
+              </friction>
+              <bounce />
+              <contact />
+            </surface>
+          </collision>
+          <visual name='visual1'>
+            <pose>0 0 ${H} 0 0 0</pose>
+            <geometry>
+              <box>
+                <size>${L} ${W} 0.03</size>
+              </box>
+            </geometry>
+            <material>
+              <diffuse>1 1 1 1</diffuse>
+              <script>
               <uri>file://media/materials/scripts/gazebo.material</uri>
               <name>Gazebo/Wood</name>
             </script>
-            <pbr>
-              <metal>
-                <albedo_map>
-                  https://fuel.gazebosim.org/1.0/openrobotics/models/table/4/files/Table_Diffuse.jpg</albedo_map>
-              </metal>
-            </pbr>
-          </material>
-        </visual>
-        <collision name='front_left_leg'>
-          <pose>0.68000000000000005 0.38 0.5 0 0 0</pose>
-          <geometry>
-            <cylinder>
-              <radius>0.02</radius>
-              <length>1</length>
-            </cylinder>
-          </geometry>
-          <surface>
-            <friction>
-              <ode />
-            </friction>
-            <bounce />
-            <contact />
-          </surface>
-        </collision>
-        <visual name='front_left_leg'>
-          <pose>0.68000000000000005 0.38 0.5 0 0 0</pose>
-          <geometry>
-            <cylinder>
-              <radius>0.02</radius>
-              <length>1</length>
-            </cylinder>
-          </geometry>
-          <material>
-            <diffuse>0.5 0.5 0.5 1</diffuse>
-            <script>
+              <pbr>
+                <metal>
+                  <albedo_map>
+                    https://fuel.gazebosim.org/1.0/openrobotics/models/table/4/files/Table_Diffuse.jpg</albedo_map>
+                </metal>
+              </pbr>
+            </material>
+          </visual>
+          <collision name='front_left_leg'>
+            <pose>${L/2 - 0.05} ${W/2 - 0.05} ${H/2} 0 0 0</pose>
+            <geometry>
+              <cylinder>
+                <radius>0.02</radius>
+                <length>${H}</length>
+              </cylinder>
+            </geometry>
+            <surface>
+              <friction>
+                <ode />
+              </friction>
+              <bounce />
+              <contact />
+            </surface>
+          </collision>
+          <visual name='front_left_leg'>
+            <pose>${L/2 - 0.05} ${W/2 - 0.05} ${H/2} 0 0 0</pose>
+            <geometry>
+              <cylinder>
+                <radius>0.02</radius>
+                <length>${H}</length>
+              </cylinder>
+            </geometry>
+            <material>
+              <diffuse>0.5 0.5 0.5 1</diffuse>
+              <script>
               <uri>file://media/materials/scripts/gazebo.material</uri>
               <name>Gazebo/Grey</name>
             </script>
-          </material>
-        </visual>
-        <collision name='front_right_leg'>
-          <pose>0.68000000000000005 -0.38 0.5 0 0 0</pose>
-          <geometry>
-            <cylinder>
-              <radius>0.02</radius>
-              <length>1</length>
-            </cylinder>
-          </geometry>
-          <surface>
-            <friction>
-              <ode />
-            </friction>
-            <bounce />
-            <contact />
-          </surface>
-        </collision>
-        <visual name='front_right_leg'>
-          <pose>0.68000000000000005 -0.38 0.5 0 0 0</pose>
-          <geometry>
-            <cylinder>
-              <radius>0.02</radius>
-              <length>1</length>
-            </cylinder>
-          </geometry>
-          <material>
-            <diffuse>0.5 0.5 0.5 1</diffuse>
-            <script>
+            </material>
+          </visual>
+          <collision name='front_right_leg'>
+            <pose>${L/2 - 0.05} -${W/2 - 0.05} ${H/2} 0 0 0</pose>
+            <geometry>
+              <cylinder>
+                <radius>0.02</radius>
+                <length>${H}</length>
+              </cylinder>
+            </geometry>
+            <surface>
+              <friction>
+                <ode />
+              </friction>
+              <bounce />
+              <contact />
+            </surface>
+          </collision>
+          <visual name='front_right_leg'>
+            <pose>${L/2 - 0.05} -${W/2 - 0.05} ${H/2} 0 0 0</pose>
+            <geometry>
+              <cylinder>
+                <radius>0.02</radius>
+                <length>${H}</length>
+              </cylinder>
+            </geometry>
+            <material>
+              <diffuse>0.5 0.5 0.5 1</diffuse>
+              <script>
               <uri>file://media/materials/scripts/gazebo.material</uri>
               <name>Gazebo/Grey</name>
             </script>
-          </material>
-        </visual>
-        <collision name='back_right_leg'>
-          <pose>-0.68000000000000005 -0.38 0.5 0 0 0</pose>
-          <geometry>
-            <cylinder>
-              <radius>0.02</radius>
-              <length>1</length>
-            </cylinder>
-          </geometry>
-          <surface>
-            <friction>
-              <ode />
-            </friction>
-            <bounce />
-            <contact />
-          </surface>
-        </collision>
-        <visual name='back_right_leg'>
-          <pose>-0.68000000000000005 -0.38 0.5 0 0 0</pose>
-          <geometry>
-            <cylinder>
-              <radius>0.02</radius>
-              <length>1</length>
-            </cylinder>
-          </geometry>
-          <material>
-            <diffuse>0.5 0.5 0.5 1</diffuse>
-            <script>
+            </material>
+          </visual>
+          <collision name='back_right_leg'>
+            <pose>-${L/2 - 0.05} -${W/2 - 0.05} ${H/2} 0 0 0</pose>
+            <geometry>
+              <cylinder>
+                <radius>0.02</radius>
+                <length>${H}</length>
+              </cylinder>
+            </geometry>
+            <surface>
+              <friction>
+                <ode />
+              </friction>
+              <bounce />
+              <contact />
+            </surface>
+          </collision>
+          <visual name='back_right_leg'>
+            <pose>-${L/2 - 0.05} -${W/2 - 0.05} ${H/2} 0 0 0</pose>
+            <geometry>
+              <cylinder>
+                <radius>0.02</radius>
+                <length>${H}</length>
+              </cylinder>
+            </geometry>
+            <material>
+              <diffuse>0.5 0.5 0.5 1</diffuse>
+              <script>
               <uri>file://media/materials/scripts/gazebo.material</uri>
               <name>Gazebo/Grey</name>
             </script>
-          </material>
-        </visual>
-        <collision name='back_left_leg'>
-          <pose>-0.68000000000000005 0.38 0.5 0 0 0</pose>
-          <geometry>
-            <cylinder>
-              <radius>0.02</radius>
-              <length>1</length>
-            </cylinder>
-          </geometry>
-          <surface>
-            <friction>
-              <ode />
-            </friction>
-            <bounce />
-            <contact />
-          </surface>
-        </collision>
-        <visual name='back_left_leg'>
-          <pose>-0.68000000000000005 0.38 0.5 0 0 0</pose>
-          <geometry>
-            <cylinder>
-              <radius>0.02</radius>
-              <length>1</length>
-            </cylinder>
-          </geometry>
-          <material>
-            <diffuse>0.5 0.5 0.5 1</diffuse>
-            <script>
+            </material>
+          </visual>
+          <collision name='back_left_leg'>
+            <pose>-${L/2 - 0.05} ${W/2 - 0.05} ${H/2} 0 0 0</pose>
+            <geometry>
+              <cylinder>
+                <radius>0.02</radius>
+                <length>${H}</length>
+              </cylinder>
+            </geometry>
+            <surface>
+              <friction>
+                <ode />
+              </friction>
+              <bounce />
+              <contact />
+            </surface>
+          </collision>
+          <visual name='back_left_leg'>
+            <pose>-${L/2 - 0.05} ${W/2 - 0.05} ${H/2} 0 0 0</pose>
+            <geometry>
+              <cylinder>
+                <radius>0.02</radius>
+                <length>${H}</length>
+              </cylinder>
+            </geometry>
+            <material>
+              <diffuse>0.5 0.5 0.5 1</diffuse>
+              <script>
               <uri>file://media/materials/scripts/gazebo.material</uri>
               <name>Gazebo/Grey</name>
             </script>
-          </material>
-        </visual>
-        <pose>0 0 0 0 0 0</pose>
-        <inertial>
+            </material>
+          </visual>
           <pose>0 0 0 0 0 0</pose>
-          <mass>1</mass>
-          <inertia>
-            <ixx>1</ixx>
-            <ixy>0</ixy>
-            <ixz>0</ixz>
-            <iyy>1</iyy>
-            <iyz>0</iyz>
-            <izz>1</izz>
-          </inertia>
-        </inertial>
-        <enable_wind>false</enable_wind>
-      </link>
-      <pose>0 0 0 0 0 1.5707900000000004</pose>
-      <self_collide>false</self_collide>
-    </model>
-    <model name='Table_0'>
-      <static>true</static>
-      <link name='link'>
-        <collision name='surface'>
-          <pose>0 0 1 0 0 0</pose>
-          <geometry>
-            <box>
-              <size>1.5 0.80000000000000004 0.029999999999999999</size>
-            </box>
-          </geometry>
-          <surface>
-            <friction>
-              <ode>
-                <mu>0.59999999999999998</mu>
-                <mu2>0.59999999999999998</mu2>
-              </ode>
-            </friction>
-            <bounce />
-            <contact />
-          </surface>
-        </collision>
-        <visual name='visual1'>
-          <pose>0 0 1 0 0 0</pose>
-          <geometry>
-            <box>
-              <size>1.5 0.80000000000000004 0.029999999999999999</size>
-            </box>
-          </geometry>
-          <material>
-            <diffuse>1 1 1 1</diffuse>
-            <script>
-              <uri>file://media/materials/scripts/gazebo.material</uri>
-              <name>Gazebo/Wood</name>
-            </script>
-            <pbr>
-              <metal>
-                <albedo_map>
-                  https://fuel.gazebosim.org/1.0/openrobotics/models/table/4/files/Table_Diffuse.jpg</albedo_map>
-              </metal>
-            </pbr>
-          </material>
-        </visual>
-        <collision name='front_left_leg'>
-          <pose>0.68000000000000005 0.38 0.5 0 0 0</pose>
-          <geometry>
-            <cylinder>
-              <radius>0.02</radius>
-              <length>1</length>
-            </cylinder>
-          </geometry>
-          <surface>
-            <friction>
-              <ode />
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